Commit message: Movement that doesn't break

File: tars.urdf (robot description, URDF)
Before this commit: robot tars, 9 links, 8 joints
Links:
- link leftleftshuttle: geometry visual box size=0.12 0.12 0.12
- link leftshuttle: geometry visual box size=0.12 0.12 0.12
- link rightrightshuttle: geometry visual box size=0.12 0.12 0.12
- link rightshuttle: geometry visual box size=0.12 0.12 0.12
- link spine: geometry visual box size=0.05 0.05 .7

Commit message: More plotting

File: tars.urdf (robot description, URDF)
Before this commit: robot tars, 9 links, 8 joints
Joints:
- joint leftleftshuttle: limit effort=10000 velocity=1 -> effort=10000 velocity=10
- joint leftshuttle: limit effort=10000 velocity=1 -> effort=10000 velocity=10
- joint rightrightshuttle: limit effort=10000 velocity=1 -> effort=10000 velocity=10
- joint rightshuttle: limit effort=10000 velocity=1 -> effort=10000 velocity=10
